Commit message: update

File: assets/unitree_description/urdf/g1/main_with_hand_new.urdf (robot description, URDF)
Before this commit: robot g1, 63 links, 62 joints
Links:
- link left_hand_base_link: geometry collision mesh filename=../hand/left_hand/meshes/hand_base_link.STL; visual mesh filename=../hand/left_hand/meshes/hand_base_link.STL
- link left_index_distal: geometry collision mesh filename=../hand/left_hand/meshes/index_distal.STL; visual mesh filename=../hand/left_hand/meshes/index_distal.STL
- link left_index_proximal: geometry collision mesh filename=../hand/left_hand/meshes/index_proximal.STL; visual mesh filename=../hand/left_hand/meshes/index_proximal.STL
- link left_middle_distal: geometry collision mesh filename=../hand/left_hand/meshes/middle_distal.STL; visual mesh filename=../hand/left_hand/meshes/middle_distal.STL
- link left_middle_proximal: geometry collision mesh filename=../hand/left_hand/meshes/middle_proximal.STL; visual mesh filename=../hand/left_hand/meshes/middle_proximal.STL
- link left_pinky_distal: geometry collision mesh filename=../hand/left_hand/meshes/pinky_distal.STL; visual mesh filename=../hand/left_hand/meshes/pinky_distal.STL
- link left_pinky_proximal: geometry collision mesh filename=../hand/left_hand/meshes/pinky_proximal.STL; visual mesh filename=../hand/left_hand/meshes/pinky_proximal.STL
- link left_ring_distal: geometry collision mesh filename=../hand/left_hand/meshes/ring_distal.STL; visual mesh filename=../hand/left_hand/meshes/ring_distal.STL
- link left_ring_proximal: geometry collision mesh filename=../hand/left_hand/meshes/ring_proximal.STL; visual mesh filename=../hand/left_hand/meshes/ring_proximal.STL
- link left_thumb_distal: geometry collision mesh filename=../hand/left_hand/meshes/thumb_distal.STL; visual mesh filename=../hand/left_hand/meshes/thumb_distal.STL
- link left_thumb_metacarpals: geometry collision mesh filename=../hand/left_hand/meshes/thumb_metacarpals.STL; visual mesh filename=../hand/left_hand/meshes/thumb_metacarpals.STL
- link left_thumb_metacarpals_base2: geometry collision mesh filename=../hand/left_hand/meshes/thumb_metacarpals_base2.STL; visual mesh filename=../hand/left_hand/meshes/thumb_metacarpals_base2.STL
- link right_hand_base_link: geometry collision mesh filename=../hand/right_hand/meshes/hand_base_link.STL; visual mesh filename=../hand/right_hand/meshes/hand_base_link.STL
- link right_index_distal: geometry collision mesh filename=../hand/right_hand/meshes/index_distal.STL; visual mesh filename=../hand/right_hand/meshes/index_distal.STL
- link right_index_proximal: geometry collision mesh filename=../hand/right_hand/meshes/index_proximal.STL; visual mesh filename=../hand/right_hand/meshes/index_proximal.STL
- link right_middle_distal: geometry collision mesh filename=../hand/right_hand/meshes/middle_distal.STL; visual mesh filename=../hand/right_hand/meshes/middle_distal.STL
- link right_middle_proximal: geometry collision mesh filename=../hand/right_hand/meshes/middle_proximal.STL; visual mesh filename=../hand/right_hand/meshes/middle_proximal.STL
- link right_pinky_distal: geometry collision mesh filename=../hand/right_hand/meshes/pinky_distal.STL; visual mesh filename=../hand/right_hand/meshes/pinky_distal.STL
- link right_pinky_proximal: geometry collision mesh filename=../hand/right_hand/meshes/pinky_proximal.STL; visual mesh filename=../hand/right_hand/meshes/pinky_proximal.STL
- link right_ring_distal: geometry collision mesh filename=../hand/right_hand/meshes/ring_distal.STL; visual mesh filename=../hand/right_hand/meshes/ring_distal.STL
- link right_ring_proximal: geometry collision mesh filename=../hand/right_hand/meshes/ring_proximal.STL; visual mesh filename=../hand/right_hand/meshes/ring_proximal.STL
- link right_thumb_distal: geometry collision mesh filename=../hand/right_hand/meshes/thumb_distal.STL; visual mesh filename=../hand/right_hand/meshes/thumb_distal.STL
- link right_thumb_metacarpals: geometry collision mesh filename=../hand/right_hand/meshes/thumb_metacarpals.STL; visual mesh filename=../hand/right_hand/meshes/thumb_metacarpals.STL
- link right_thumb_metacarpals_base2: geometry collision mesh filename=../hand/right_hand/meshes/thumb_metacarpals_base2.STL; visual mesh filename=../hand/right_hand/meshes/thumb_metacarpals_base2.STL
